File: Electrical/Light_Project/pcb_layout_light.brd (EAGLE design)
At the start: 27.9 x 20 mm, 12 parts, among them U1 REG710NA-3.3/3K, U2 ATTINY85V-10SU, U3 FSM8JRT

Commit message: Add BOM
Connections:
- removed net N$4: C3.2, U1.3, U1.5
- net GND: now also C3.2
- net N$8: now also U1.3, U1.5
Routing:
- net GND: track 36.7 -> 64.8 mm
- net N$8: track 2.11 -> 8.95 mm
- net N$4: track 5.52 -> 0.00 mm
Changed lines of the file:
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@@
 <contactref element="JP2" pad="1"/>
 <wire x1="29.21" y1="13.97" x2="34.29" y2="13.97" width="0.3048" layer="1"/>
-<wire x1="34.29" y1="4.9276" x2="34.29" y2="5.08" width="0" layer="19" extent="1-1"/>
+<contactref element="C3" pad="2"/>
+<wire x1="30.91" y1="3.81" x2="33.02" y2="-1.27" width="0.3048" layer="1"/>
+<wire x1="33.02" y1="-1.27" x2="43.18" y2="-1.27" width="0.3048" layer="1"/>
+<wire x1="43.18" y1="-1.27" x2="45.72" y2="2.54" width="0.3048" layer="1"/>
+<wire x1="45.72" y1="2.54" x2="46.99" y2="8.89" width="0.3048" layer="1"/>
+<wire x1="46.99" y1="8.89" x2="45.72" y2="9.3916" width="0.3048" layer="1"/>
+<wire x1="34.29" y1="5.08" x2="34.29" y2="4.9276" width="0" layer="19" extent="1-1"/>
 </signal>
 <signal name="N$1">
@@
 <wire x1="35.24" y1="4.9276" x2="35.56" y2="6.35" width="0.3048" layer="1"/>
 <wire x1="35.56" y1="6.35" x2="34.72" y2="7.62" width="0.3048" layer="1"/>
-</signal>
-<signal name="N$4">
-<contactref element="U1" pad="5"/>
-<contactref element="U1" pad="3"/>
-<contactref element="C3" pad="2"/>
-<wire x1="30.91" y1="3.81" x2="32.0276" y2="4.9276" width="0.3048" layer="1"/>
-<wire x1="32.0276" y1="4.9276" x2="33.34" y2="4.9276" width="0.3048" layer="1"/>
-<wire x1="33.34" y1="4.9276" x2="33.7058" y2="4.5618" width="0.3048" layer="1"/>
-<wire x1="33.9242" y1="3.55525" x2="33.9242" y2="3.0582" width="0.3048" layer="1"/>
-<wire x1="33.9242" y1="3.0582" x2="34.29" y2="2.6924" width="0.3048" layer="1"/>
-<wire x1="33.7058" y1="4.5618" x2="33.7058" y2="3.77365" width="0.3048" layer="1"/>
-<wire x1="33.7058" y1="3.77365" x2="33.9242" y2="3.55525" width="0.3048" layer="1"/>
 </signal>
 <signal name="N$5">
@@
 <wire x1="34.4816" y1="12.065" x2="35.6743" y2="12.065" width="0.3048" layer="1"/>
 </signal>
-<signal name="N$8">
-<contactref element="C3" pad="1"/>
-<contactref element="JP1" pad="3"/>
-<wire x1="27.94" y1="3.81" x2="30.05" y2="3.81" width="0.3048" layer="1"/>
-</signal>
 <signal name="N$10">
 <contactref element="JP2" pad="2"/>
@@
 <wire x1="25.4" y1="10.16" x2="26.67" y2="13.97" width="0.3048" layer="1"/>
 </signal>
+<signal name="N$8">
+<contactref element="C3" pad="1"/>
+<contactref element="JP1" pad="3"/>
+<contactref element="U1" pad="5"/>
+<contactref element="U1" pad="3"/>
+<wire x1="32.0276" y1="4.9276" x2="33.34" y2="4.9276" width="0.3048" layer="1"/>
+<wire x1="33.34" y1="4.9276" x2="33.7058" y2="4.5618" width="0.3048" layer="1"/>
+<wire x1="33.9242" y1="3.55525" x2="33.9242" y2="3.0582" width="0.3048" layer="1"/>
+<wire x1="33.9242" y1="3.0582" x2="34.29" y2="2.6924" width="0.3048" layer="1"/>
+<wire x1="33.7058" y1="4.5618" x2="33.7058" y2="3.77365" width="0.3048" layer="1"/>
+<wire x1="33.7058" y1="3.77365" x2="33.9242" y2="3.55525" width="0.3048" layer="1"/>
+<wire x1="27.94" y1="3.81" x2="30.05" y2="3.81" width="0.3048" layer="1"/>
+<wire x1="30.05" y1="3.81" x2="30.48" y2="5.08" width="0.3048" layer="1"/>
+<wire x1="30.48" y1="5.08" x2="32.0276" y2="4.9276" width="0.3048" layer="1"/>
+</signal>
 </signals>
